File: code/streamdeck-vu-driver.kicad_sch (KiCad schematic)
At the start: 7 parts, among them J1 Pi_SPI0, U1 MCP4922

Commit message: v0.3.1 — rename project to TheStreamDeck
Renamed from "StreamDeck Pi" to "TheStreamDeck". Directory moved from
PROJECTS/private/streaming-appliance/ to PROJECTS/public/TheStreamDeck/.
All references updated across specs, diagrams, KiCad schematic, LaTeX
sources, and PAI memory index.
Other:
- note added: "THESTREAMDECK - VU METER DRIVER"
- note removed: "STREAMDECK PI - VU METER DRIVER"
- title: StreamDeck Pi - VU Meter Driver -> TheStreamDeck - VU Meter Driver
Changed lines of the file:
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@@
 	(paper "A4")
 	(title_block
-		(title "StreamDeck Pi - VU Meter Driver")
+		(title "TheStreamDeck - VU Meter Driver")
 		(date "2026-04-05")
 		(rev "A")
@@
 		(stroke (width 0) (type solid))
 	)
-	(text "STREAMDECK PI - VU METER DRIVER"
+	(text "THESTREAMDECK - VU METER DRIVER"
 		(exclude_from_sim no)
 		(at 25 15 0)
